File: corne-ice/pcb/corne-ice.kicad_pcb (KiCad board)
At the start: 2 copper layers, 275.5 x 105.6 mm, 120 parts, among them J1 BAT, J2 nice!view, J3 BAT, J4 nice!view, SW1 SW_PUSH, SW10 SW_PUSH, SW11 SW_PUSH, SW12 SW_PUSH, SW13 SW_PUSH, SW14 SW_PUSH, SW15 SW_PUSH, SW16 SW_PUSH, SW17 SW_PUSH, SW18 SW_PUSH, SW19 SW_PUSH, SW2 SW_PUSH, SW20 SW_PUSH, SW21 SW_PUSH, SW22 SW_PUSH, SW23 SW_PUSH, SW24 SW_PUSH, SW25 SW_PUSH, SW26 SW_PUSH, SW27 SW_PUSH, SW28 SW_PUSH, SW29 SW_PUSH, SW3 SW_PUSH, SW30 SW_PUSH, SW31 SW_PUSH, SW32 SW_PUSH, SW33 SW_PUSH, SW34 SW_PUSH, SW35 SW_PUSH, SW36 SW_PUSH, SW37 SW_PUSH, SW38 SW_PUSH, SW39 SW_PUSH, SW4 SW_PUSH, SW40 SW_PUSH, SW41 SW_PUSH, SW42 SW_PUSH, SW5 SW_PUSH, SW6 SW_PUSH, SW7 SW_PUSH, SW8 SW_PUSH, SW9 SW_PUSH, U1 nice!nano, U2 nice!nano

Commit message: Added a button and rotary encoder.
Parts:
- removed G*** (x4): LOGO, kbd:corne-logo-horizontal
- removed J1: BAT, Connector_JST:JST_PH_S2B-PH-SM4-TB_1x02-1MP_P2.00mm_Horizontal
- removed J2: nice!view, Connector_PinHeader_2.54mm:PinHeader_1x05_P2.54mm_Vertical
- removed REF** (x8): Breakaway_Tabs, kbd:Breakaway_Tabs
- removed RST: SW_PUSH, keeblib:alps_sksn
- removed Ref** (x14): Val**, kbd:M2_HOLE_v2
- added D43: D, kbd:D3_SMD_v2, B.Cu at (75.1, 88.5)
- added RSW1: SW_PUSH, Button_Switch_SMD:SW_Push_1P1T-MP_NO_Horizontal_Alps_SKRTLAE010, F.Cu at (142.8, 63.9)
- added SW43: RotaryEncoder_Switch, Rotary_Encoder:RotaryEncoder_Alps_EC11E-Switch_Vertical_H20mm, F.Cu at (126.7, 68.1)
- added SW44: SW_PUSH, kbd:CherryMX_Hotswap, F.Cu at (67.5, 88.7)
- added TP1: TestPoint, TestPoint:TestPoint_Pad_1.5x1.5mm, F.Cu at (130.6, 63.5)
- added TP2: TestPoint, TestPoint:TestPoint_Pad_D1.5mm, F.Cu at (127.3, 63.5)
- PSW1: value POWER -> SW_SPDT; moved to F.Cu
- PSW2: value POWER -> SW_SPDT
- moved PSW1 52.7 mm to (143.0, 80.7), turned to 90 degrees
- moved D20 23.3 mm to (118.4, 90.9)
- moved D21 23.3 mm to (121.2, 90.9)
- moved D19 18.7 mm to (94.8, 88.5)
- renumbered RST to RSW2
Routing:
- net row1: track 191.4 -> 124.9 mm
- net RAW: track 5.71 -> 58.7 mm, vias 0 -> 1
- net row2: track 181.3 -> 136.4 mm
- net Net-(PSW1-B): track 66.2 -> 22.7 mm, vias 1 -> 0
- net row0: track 169.1 -> 127.1 mm
- net VCC: track 37.8 -> 0.00 mm
- net CS: track 37.3 -> 0.00 mm
- net MOSI: track 33.6 -> 0.00 mm
- net Net-(D21-A): track 38.3 -> 7.81 mm
- net col2: track 125.8 -> 155.6 mm, vias 5 -> 4
- net SCK: track 28.9 -> 0.00 mm
- net row3: track 122.5 -> 101.2 mm
- net Net-(D20-A): track 23.7 -> 4.30 mm
- net Net-(D19-A): track 22.2 -> 4.11 mm
- net GND: track 70.1 -> 56.1 mm
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Other:
- board size 275.5 x 105.6 mm -> 274.3 x 91.5 mm
