File: corne-ice/pcb/corne-ice.kicad_sch (KiCad schematic)
At the start: 97 parts, among them J3 BAT, J4 nice!view, SW1 SW_PUSH, SW10 SW_PUSH, SW11 SW_PUSH, SW12 SW_PUSH, SW13 SW_PUSH, SW14 SW_PUSH, SW15 SW_PUSH, SW16 SW_PUSH, SW17 SW_PUSH, SW18 SW_PUSH, SW19 SW_PUSH, SW2 SW_PUSH, SW20 SW_PUSH, SW21 SW_PUSH, SW22 SW_PUSH, SW23 SW_PUSH, SW24 SW_PUSH, SW25 SW_PUSH, SW26 SW_PUSH, SW27 SW_PUSH, SW28 SW_PUSH, SW29 SW_PUSH, SW3 SW_PUSH, SW30 SW_PUSH, SW31 SW_PUSH, SW32 SW_PUSH, SW33 SW_PUSH, SW34 SW_PUSH, SW35 SW_PUSH, SW36 SW_PUSH, SW37 SW_PUSH, SW38 SW_PUSH, SW39 SW_PUSH, SW4 SW_PUSH, SW40 SW_PUSH, SW41 SW_PUSH, SW42 SW_PUSH, SW43 RotaryEncoder_Switch, SW44 SW_PUSH, SW5 SW_PUSH, SW6 SW_PUSH, SW7 SW_PUSH, SW8 SW_PUSH, SW9 SW_PUSH, U1 nice!nano, U2 nice!nano

Commit message: Left part updated
Parts:
- removed D10, D11, D12, D13, D14, D15, D16, D17, D18, D19, D20, D21, D43, D7, D8, D9: D, kbd:D3_SMD_v2, symbol Device:D
- removed SW10, SW11, SW12, SW13, SW14, SW15, SW16, SW17, SW18, SW19, SW20, SW44, SW6, SW7, SW8, SW9: SW_PUSH, kbd:CherryMX_Hotswap, symbol kbd:SW_PUSH
- removed SW21: SW_PUSH, kbd:CherryMX_Hotswap_1.5u, symbol kbd:SW_PUSH
- added D44, D45, D46, D47, D48, D49, D50, D51, D52, D53, D54, D55, D56, D57, D58, D59, D60: D, kbd:D3_SMD_v2, symbol Device:D
- added SW45, SW46, SW47, SW48, SW49, SW50, SW51, SW52, SW53, SW54, SW55, SW56, SW57, SW58, SW59, SW60, SW61: SW_PUSH, kbd:CherryMX_Hotswap, symbol kbd:SW_PUSH
- SW5: footprint kbd:CherryMX_Hotswap -> kbd:CherryMX_Hotswap_1.5u
Connections:
- net GND: now also SW43.C
- net col0: now also SW45.1, SW46.1
- net col1: now also SW43.S1, SW47.1, SW48.1, SW49.1; no longer SW2.1
- net col2: now also SW2.1, SW50.1, SW51.1, SW52.1; no longer SW3.1
- net col3: now also SW3.1, SW53.1, SW54.1, SW55.1; no longer SW4.1
- net col4: now also SW4.1, SW56.1, SW57.1, SW58.1; no longer SW5.1
- net col5: now also SW5.1, SW59.1, SW60.1, SW61.1
- net row0: now also D46.1 (K), D49.1 (K), D52.1 (K), D55.1 (K), D58.1 (K); no longer D2.1 (K), D3.1 (K), D4.1 (K), D5.1 (K), D6.1 (K)
- net row1: now also D44.1 (K), D47.1 (K), D50.1 (K), D53.1 (K), D56.1 (K), D59.1 (K)
- net row2: now also D45.1 (K), D48.1 (K), D51.1 (K), D54.1 (K), D57.1 (K), D60.1 (K)
- net row3: now also D2.1 (K), D3.1 (K), D4.1 (K), D5.1 (K), D6.1 (K)
- net rotary_a: now reaches U1.13 (NFC1/P0.09)
- net rotary_a: now also SW43.A
- net rotary_b: now reaches U1.14 (NFC2/P0.10)
- net rotary_b: now also SW43.B
- net at D6.2 (A): now also SW43.S2
- new net: D51.2 (A), SW52.2
- new net: D56.2 (A), SW57.2
- new net: D46.2 (A), SW47.2
- new net: D54.2 (A), SW55.2
- new net: D49.2 (A), SW50.2
- new net: D50.2 (A), SW51.2
- new net: D48.2 (A), SW49.2
- new net: D53.2 (A), SW54.2
- new net: D57.2 (A), SW58.2
- new net: D52.2 (A), SW53.2
- new net: D58.2 (A), SW59.2
- new net: D55.2 (A), SW56.2
- new net: D44.2 (A), SW45.2
- new net: D45.2 (A), SW46.2
- new net: D47.2 (A), SW48.2
- new net: D60.2 (A), SW61.2
- new net: D59.2 (A), SW60.2
- no-connect marks 18 -> 16
Other:
- moved on the sheet: D1, PSW1, RSW1, SW1, SW43, TP1, TP2, U1

Commit message: Right half
Parts:
- removed J3: BAT, Connector_JST:JST_PH_S2B-PH-SM4-TB_1x02-1MP_P2.00mm_Horizontal, symbol Connector_Generic:Conn_01x02
- removed J4: nice!view, Connector_PinHeader_2.54mm:PinHeader_1x05_P2.54mm_Vertical, symbol Connector_Generic:Conn_01x05
- added D7, D8: D, kbd:D3_SMD_v2, symbol Device:D
- added RSW3: SW_PUSH, Button_Switch_SMD:SW_Push_1P1T-MP_NO_Horizontal_Alps_SKRTLAE010, symbol kbd:SW_PUSH
- added SW6: SW_PUSH, kbd:CherryMX_Hotswap, symbol kbd:SW_PUSH
- added SW7: RotaryEncoder_Switch, Rotary_Encoder:RotaryEncoder_Alps_EC11E-Switch_Vertical_H20mm, symbol Device:RotaryEncoder_Switch
- added TP3: TestPoint, TestPoint:TestPoint_Pad_D1.5mm, symbol Connector:TestPoint
- added TP4: TestPoint, TestPoint:TestPoint_Pad_1.5x1.5mm, symbol Connector:TestPoint
Connections:
- net GNDA: now also RSW3.2, SW7.C, TP4.1
- net col1_r: now also SW7.S1
- net col2_r: now also SW6.1
- net reset_r: now also RSW3.1
- net row3_r: now also D7.1 (K), D8.1 (K)
- net rotary_a_r: now reaches U2.13 (NFC1/P0.09)
- net rotary_a_r: now also SW7.A
- net rotary_b_r: now reaches U2.14 (NFC2/P0.10)
- net rotary_b_r: now also SW7.B
- net at PSW2.2 (B): now also TP3.1
- new net: D7.2 (A), SW6.2
- new net: D8.2 (A), SW7.S2
- no-connect marks 16 -> 14
Other:
- moved on the sheet: D1, D2, D22, D23, D24, D25, D26, D27, D28, D29, D3, D30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

Commit message: Backup.
Changed lines of the file:
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@@
-    )
-  )
-  (global_label "reset_r" (shape input) (at 69.85 138.43 180) (fields_autoplaced)
-    (effects (font (size 1.524 1.524)) (justify right))
-    (property "Intersheetrefs" "${INTERSHEET_REFS}" (at 59.2881 138.43 0)
-      (effects (font (size 1.27 1.27)) (justify right) hide)
     )
   )
@@
       (effects (font (size 1.27 1.27)) (justify right) hide)
     )
+  )
+  (global_label "reset_r" (shape input) (at 69.85 138.43 180) (fields_autoplaced)
+    (effects (font (size 1.1938 1.1938)) (justify right))
+    (property "Intersheetrefs" "${INTERSHEET_REFS}" (at 61.5763 138.43 0)
+      (effects (font (size 1.27 1.27)) (justify right) hide)
+    )

Commit message: Ordered.
Parts:
- removed RSW3: SW_PUSH, Button_Switch_SMD:SW_Push_1P1T-MP_NO_Horizontal_Alps_SKRTLAE010, symbol kbd:SW_PUSH
- RSW1: value SW_PUSH -> CPG151101S11-16; footprint Button_Switch_SMD:SW_Push_1P1T-MP_NO_Horizontal_Alps_SKRTLAE010 -> kbd:CherryMX_Hotswap; symbol kbd:SW_PUSH -> jlc_pcb:switch_socket
- RSW2: value SW_PUSH -> CPG151101S11-16; footprint keeblib:alps_sksn -> kbd:CherryMX_Hotswap; symbol kbd:SW_PUSH -> jlc_pcb:switch_socket
- SW1, SW2, SW22, SW23, SW24, SW25, SW26, SW27, SW28, SW29, SW3, SW30, SW31, SW32, SW33, SW34, SW35, SW36, SW37, SW38, SW39, SW4, SW40, SW41, SW45, SW46, SW47, SW48, SW49, SW50, SW51, SW52, SW53, SW54, SW55, SW56, SW57, SW58, SW59, SW6, SW60, SW61: value SW_PUSH -> CPG151101S11-16; symbol kbd:SW_PUSH -> jlc_pcb:switch_socket
- SW42, SW5: value SW_PUSH -> CPG151101S11-16; footprint kbd:CherryMX_Hotswap_1.5u -> kbd:CherryMX_Hotswap; symbol kbd:SW_PUSH -> jlc_pcb:switch_socket_1.5
